Commit message: should be able to use tiny renderer now

File: stirring/urdf/cup/invisible_cup_small.urdf (robot description, URDF)
Before this commit: robot cube.urdf, 1 links, 0 joints
Links:
- link baseLink: geometry collision mesh filename=Cup/cup_vhacd.obj scale=0.5 0.5 0.5; visual mesh filename=Cup/textured-0008192.obj scale=0.5 0.5 0.5
