Commit message: made spheres heavier, added scaling factor

File: stirring/urdf/cup/cup_small.urdf (robot description, URDF)
Before this commit: robot cube.urdf, 1 links, 0 joints
Links:
- link baseLink: mass 3.5 -> 10.5

File: stirring/urdf/invisible_plane.urdf (robot description, URDF)
Before this commit: robot plane, 1 links, 0 joints
Links:
- link planeLink: mass .0 -> 0.0

File: stirring/urdf/sphere/blue_sphere.urdf (robot description, URDF)
Before this commit: robot urdf_robot, 1 links, 0 joints
Links:
- link baseLink: mass 1.0 -> 0.1

File: stirring/urdf/sphere/red_sphere.urdf (robot description, URDF)
Before this commit: robot urdf_robot, 1 links, 0 joints
Links:
- link baseLink: mass 1.0 -> 0.08

Commit message: improved reward function, and made it the change in mixed state

File: stirring/urdf/cup/cup_small.urdf (robot description, URDF)
Before this commit: robot cube.urdf, 1 links, 0 joints
Links:
- link baseLink: mass 10.5 -> 20.5

File: stirring/urdf/sphere/blue_sphere.urdf (robot description, URDF)
Before this commit: robot urdf_robot, 1 links, 0 joints
Links:
- link baseLink: mass 0.3 -> 0.1

File: stirring/urdf/sphere/red_sphere.urdf (robot description, URDF)
Before this commit: robot urdf_robot, 1 links, 0 joints
Links:
- link baseLink: mass 0.4 -> 0.1

Commit message: harder problem

File: stirring/urdf/cup/cup_small.urdf (robot description, URDF)
Before this commit: robot cube.urdf, 1 links, 0 joints
Links:
- link baseLink: mass 20.5 -> 15.5

File: stirring/urdf/sphere/blue_sphere.urdf (robot description, URDF)
Before this commit: robot urdf_robot, 1 links, 0 joints
Links:
- link baseLink: mass 0.1 -> 0.05

File: stirring/urdf/sphere/red_sphere.urdf (robot description, URDF)
Before this commit: robot urdf_robot, 1 links, 0 joints
Links:
- link baseLink: mass 0.1 -> 0.05

Commit message: heavier cup and spheres

File: stirring/urdf/cup/cup_small.urdf (robot description, URDF)
Before this commit: robot cube.urdf, 1 links, 0 joints
Links:
- link baseLink: mass 15.5 -> 60.5

File: stirring/urdf/sphere/blue_sphere.urdf (robot description, URDF)
Before this commit: robot urdf_robot, 1 links, 0 joints
Links:
- link baseLink: mass 0.05 -> 0.4

File: stirring/urdf/sphere/red_sphere.urdf (robot description, URDF)
Before this commit: robot urdf_robot, 1 links, 0 joints
Links:
- link baseLink: mass 0.05 -> 0.4
