Commit message: added beads not incup to rewaard function, distance from cup

File: stirring/urdf/sphere/blue_sphere.urdf (robot description, URDF)
Before this commit: robot urdf_robot, 1 links, 0 joints
Links:
- link baseLink: mass 0.1 -> 0.3

File: stirring/urdf/sphere/red_sphere.urdf (robot description, URDF)
Before this commit: robot urdf_robot, 1 links, 0 joints
Links:
- link baseLink: mass 0.1 -> 0.4
