Commit message: made the controller stop only when it gets close

File: stirring/urdf/sphere/red_sphere.urdf (robot description, URDF)
Before this commit: robot urdf_robot, 1 links, 0 joints
Links:
- link baseLink: mass 0.08 -> 0.1

Commit message: Fixed some bugs, learns reasonably, variable force

File: stirring/urdf/sphere/red_sphere.urdf (robot description, URDF)
Before this commit: robot urdf_robot, 1 links, 0 joints
Links:
- link baseLink: mass 2 -> 0.2
