Commit message: pr2 now does the actions

File: cup_skills/urdf/cup/cup_1.urdf (robot description, URDF)
Before this commit: robot cube.urdf, 1 links, 0 joints
Links:
- link baseLink: mass 90.5 -> .9

File: cup_skills/urdf/cup/cup_4.urdf (robot description, URDF)
Before this commit: robot cup_3.urdf, 1 links, 0 joints
Links:
- link baseLink: mass 90.5 -> 40

File: cup_skills/urdf/cup/cup_small.urdf (robot description, URDF)
Before this commit: robot cube.urdf, 1 links, 0 joints
Links:
- link baseLink: mass 90.5 -> 15.5

File: cup_skills/urdf/sphere/blue_sphere.urdf (robot description, URDF)
Before this commit: robot urdf_robot, 1 links, 0 joints
Links:
- link baseLink: mass 0.1 -> .01
