Commit message: More realistic cups, chooses from them appropriately, should be good to go

File: cup_skills/urdf/cup/cup_7.urdf (robot description, URDF)
Before this commit: robot cube.urdf, 1 links, 0 joints
Links:
- link baseLink: mass .9 -> 90.5; geometry collision mesh filename=Cup/cup_vhacd.obj scale=1.4857 1.4857 0.5964; visual mesh filename=Cup/textured-0008192.obj scale=1.4857 1.4857 0.5964

File: cup_skills/urdf/cup/cup_8.urdf (robot description, URDF)
Before this commit: robot cube.urdf, 1 links, 0 joints
Links:
- link baseLink: mass .9 -> 90.5; geometry collision mesh filename=Cup/cup_vhacd.obj scale=1.257 1.257 0.378; visual mesh filename=Cup/textured-0008192.obj scale=1.257 1.257 0.378

File: cup_skills/urdf/cup/cup_9.urdf (robot description, URDF)
Before this commit: robot cube.urdf, 1 links, 0 joints
Links:
- link baseLink: mass .9 -> 90.5; geometry collision mesh filename=Cup/cup_vhacd.obj scale=1.657 1.657 0.6545; visual mesh filename=Cup/textured-0008192.obj scale=1.657 1.657 0.6545

File: cup_skills/urdf/cup/cup_pourer.urdf (robot description, URDF)
Before this commit: robot cube.urdf, 1 links, 0 joints
Links:
- link baseLink: mass .9 -> 90.5; geometry collision mesh filename=Cup/cup_vhacd.obj scale=0.777 0.777 0.756; visual mesh filename=Cup/textured-0008192.obj scale=0.777 0.777 0.756
