Commit message: trying to make this realistic...

File: cup_skills/urdf/sphere/blue_sphere.urdf (robot description, URDF)
Before this commit: robot urdf_robot, 1 links, 0 joints
Links:
- link baseLink: mass .01 -> .003; geometry collision sphere radius=0.01

File: cup_skills/urdf/sphere/red_sphere.urdf (robot description, URDF)
Before this commit: robot urdf_robot, 1 links, 0 joints
Links:
- link baseLink: mass 0.2 -> 0.003
