Commit message: recalibrated physics parameters to be more realistic

File: cup_skills/urdf/green_spoon.urdf (robot description, URDF)
Before this commit: robot green_spoon.urdf, 1 links, 0 joints
Links:
- link baseLink: mass 1.0 -> 0.3

File: cup_skills/urdf/sphere/blue_sphere.urdf (robot description, URDF)
Before this commit: robot urdf_robot, 1 links, 0 joints
Links:
- link baseLink: mass .003 -> .03

File: cup_skills/urdf/sphere/blue_sphere_old.urdf (robot description, URDF)
Before this commit: robot cube.urdf, 1 links, 0 joints
Links:
- link baseLink: mass 0.05 -> .01; geometry collision sphere radius=0.01; visual mesh filename=sphere_smooth.obj scale=0.01 0.01 0.01

File: cup_skills/urdf/sphere/red_sphere.urdf (robot description, URDF)
Before this commit: robot urdf_robot, 1 links, 0 joints
Links:
- link baseLink: mass 0.003 -> 0.03

Commit message: green spoon now has another jnt

File: cup_skills/urdf/green_spoon.urdf (robot description, URDF)
Before this commit: robot green_spoon.urdf, 1 links, 0 joints
Links:
- added link dummy
Joints:
- added joint joint: type fixed, parent baseLink, child dummy
